File: hardware/quakelight.kicad_pcb (KiCad board)
At the start: 4 copper layers, 40 x 60 mm, 64 parts, among them J1 USB_C_Receptacle_USB2.0, J10 Conn_01x02_MountingPin, J2 RJ45_Abracon_ARJP11A-MASA-B-A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, J3 EZmate-4, J4 Conn_01x03_MountingPin, J5 Conn_01x03_MountingPin, J6 Conn_01x03_MountingPin, J7 TC2030-IDC-NL, SW1 SW_Push, SW2 SW_Push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

Commit message: wip
Parts:
- removed J6: Conn_01x03_MountingPin, Connector_JST:JST_PH_S3B-PH-SM4-TB_1x03-1MP_P2.00mm_Horizontal
- removed U7: SN74LV1T125DBV, Package_TO_SOT_SMD:SOT-23-5
- added C14: 100u, Capacitor_SMD:C_1206_3216Metric, F.Cu at (155.1, 92.9)
- added C15: 100u, Capacitor_SMD:C_1206_3216Metric, F.Cu at (143.8, 92.9)
- added C16: 100u, Capacitor_SMD:C_1206_3216Metric, F.Cu at (141.7, 92.9)
- added C20: 100n, balto:C_0402_Worthington, F.Cu at (124.1, 90.7)
- added C21: 100n, balto:C_0402_Worthington, F.Cu at (146.3, 90.7)
- added C22: 100n, balto:C_0402_Worthington, F.Cu at (135.1, 90.7)
- added C23: 100u, Capacitor_SMD:C_1206_3216Metric, F.Cu at (133.7, 100.2)
- added C24: 100u, Capacitor_SMD:C_1206_3216Metric, F.Cu at (136.0, 100.2)
- added C25: 100u, Capacitor_SMD:C_1206_3216Metric, F.Cu at (131.4, 100.2)
- added D3: SMAJ58A, Diode_SMD:D_SMA, F.Cu at (135.9, 120.0)
- added J9: PH, Connector_JST:JST_PH_S4B-PH-SM4-TB_1x04-1MP_P2.00mm_Horizontal, F.Cu at (127.0, 85.5)
- added R10: 100, balto:R_0402_Worthington, F.Cu at (128.5, 93.0)
- added R11: 100, balto:R_0402_Worthington, F.Cu at (139.5, 92.0)
- added R14: 100, balto:R_0402_Worthington, F.Cu at (139.5, 93.0)
- added R15: 100, balto:R_0402_Worthington, F.Cu at (150.7, 92.0)
- added R16: 100, balto:R_0402_Worthington, F.Cu at (150.7, 93.0)
- added R6: 0, balto:R_0402_Worthington, F.Cu at (151.8, 109.5)
- added R7: 1k, balto:R_0402_Worthington, F.Cu at (146.6, 98.1)
- added R8: 100, balto:R_0402_Worthington, F.Cu at (128.5, 92.0)
- added U8: SN74LVC2T45DCUR, Package_SO:VSSOP-8_2.3x2mm_P0.5mm, F.Cu at (125.3, 92.4)
- C13, C4, C8: value 10u -> 100u; footprint balto:C_0402_Worthington -> Capacitor_SMD:C_1206_3216Metric
- C19: footprint Capacitor_SMD:CP_Elec_6.3x7.7 -> Capacitor_SMD:C_1206_3216Metric
- J4, J5: value Conn_01x03_MountingPin -> PH; footprint Connector_JST:JST_PH_S3B-PH-SM4-TB_1x03-1MP_P2.00mm_Horizontal -> Connector_JST:JST_PH_S4B-PH-SM4-TB_1x04-1MP_P2.00mm_Horizontal
- U4, U5: value SN74LV1T125DBV -> SN74LVC2T45DCUR; footprint Package_TO_SOT_SMD:SOT-23-5 -> Package_SO:VSSOP-8_2.3x2mm_P0.5mm
- moved C8 23.4 mm to (130.7, 92.9), turned to -90 degrees
- moved J4 12.0 mm to (140.0, 85.5)
- moved C10 11.8 mm to (148.7, 90.7), turned to 180 degrees
- moved C6 11.6 mm to (137.5, 90.7), turned to 180 degrees
- moved C13 11.2 mm to (153.0, 92.9), turned to -90 degrees
- moved U4 9.31 mm to (136.3, 92.4), turned to 0 degrees
- moved U5 3.52 mm to (147.5, 92.4), turned to 0 degrees
- moved C4 3.38 mm to (132.8, 92.9), turned to -90 degrees
- moved C19 3.36 mm to (138.3, 100.2), turned to 90 degrees
- moved C3 3.28 mm to (140.2, 100.3)
- moved C1 3.16 mm to (146.4, 103.2), turned to -90 degrees
- moved U1 2.20 mm to (148.8, 103.7), turned to 0 degrees
- moved FID1 2.00 mm to (122.0, 92.0)
- moved FID3 2.00 mm to (158.0, 92.0)
- moved J2 2.00 mm to (125.3, 124.0)
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Connections:
- J4 pad 3: GND -> Net-(J4-Pin_3)
- J5 pad 3: GND -> Net-(J5-Pin_3)
- SW1 pad 1: /SW1 -> /BOOT0
- SW1 pad 2: GND -> +3V3
- U10 pad 45: unconnected-(U10-PA9-Pad45) -> /SPI2_SCK
- U10 pad 54: unconnected-(U10-PC10-Pad54) -> /SPI3_SCK
- U10 pad 57: unconnected-(U10-PB3(JTDO-Pad57) -> /SPI1_SCK
- U10 pad 62: GND -> /BOOT0
- U10 pad 63: unconnected-(U10-PB8-Pad63) -> /SW1
- U4 pad 1: GND -> +3V3
- U4 pad 2: /SPI1_MOSI -> /SPI2_SCK
- U4 pad 3: GND -> /SPI2_MOSI
- U4 pad 4: Net-(J4-Pin_2) -> GND
- U4 pad 5: +5V -> +3V3
- U5 pad 1: GND -> +3V3
- U5 pad 2: /SPI2_MOSI -> /SPI3_SCK
- U5 pad 3: GND -> /SPI3_MOSI
- U5 pad 4: Net-(J5-Pin_2) -> GND
- U5 pad 5: +5V -> +3V3
Routing:
- net Net-(J6-Pin_2): track 3.03 -> 0.00 mm
- net Net-(J5-Pin_2): track 3.03 -> 0.00 mm
- net Net-(J4-Pin_2): track 3.03 -> 0.00 mm
Other:
- board size 40 x 60 mm -> 40 x 62 mm

Commit message: wip
Parts:
- added C26: 1u, balto:C_0402_Worthington, F.Cu at (143.5, 97.2)
- added C27: 1u, balto:C_0402_Worthington, F.Cu at (142.5, 100.7)
- added G***: LOGO, balto:paw_copper, F.Cu at (155.5, 132.6)
- R12: value 75k -> 36k
- R5: value 75k -> 0; footprint balto:R_0402_Worthington -> Resistor_SMD:R_0805_2012Metric
- moved R5 32.6 mm to (142.0, 131.0), turned to -90 degrees
- moved C68 12.6 mm to (129.1, 120.6), turned to 90 degrees
- moved C69 11.2 mm to (130.3, 120.6), turned to 90 degrees
- moved R7 10.8 mm to (151.6, 107.7)
- moved FID2 6.00 mm to (158.0, 140.0)
- moved R12 3.30 mm to (144.4, 100.7), turned to 0 degrees
- moved R22 2.49 mm to (142.8, 135.9), turned to 180 degrees
- moved U6 2.33 mm to (142.7, 98.9), turned to 90 degrees
- moved R13 2.16 mm to (144.4, 101.7), turned to 180 degrees
- moved R23 1.86 mm to (142.8, 136.9), turned to 180 degrees
- moved C67 1.70 mm to (144.8, 123.3), turned to 90 degrees
- moved C66 1.14 mm to (143.8, 123.3), turned to 90 degrees
- moved C59 1.03 mm to (149.3, 120.8), turned to 180 degrees
- moved C61 0.90 mm to (157.7, 111.7), turned to -90 degrees
- moved C60 0.64 mm to (155.8, 121.0), turned to 180 degrees
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Connections:
- J2 pad SH: GND -> Net-(J2-PadSH)
- R5 pad 1: +5V_DCDC -> Net-(J2-PadSH)
- R5 pad 2: Net-(U6-PR1) -> GND
- U10 pad 14: unconnected-(U10-PA0-Pad14) -> /ETH_LED_0
- U10 pad 17: /ETH_INT -> /ETH_RESET
- U10 pad 22: unconnected-(U10-PA6-Pad22) -> /ETH_INT
- U10 pad 26: unconnected-(U10-PB0-Pad26) -> /SW0
- U10 pad 27: unconnected-(U10-PB1-Pad27) -> /LED_B
- U10 pad 28: unconnected-(U10-PB2-Pad28) -> /LED_A
- U10 pad 8: /ETH_RESET -> unconnected-(U10-PC0-Pad8)
Routing:
- net GND: track 0.00 -> 73.3 mm, vias 0 -> 127
- net +3V3: track 0.00 -> 53.2 mm, vias 0 -> 22
- net /ETH_RX_N: track 0.00 -> 46.2 mm, vias 0 -> 1
- net /ETH_RX_P: track 0.00 -> 46.1 mm, vias 0 -> 1
- net /ETH_TX_N: track 0.00 -> 45.9 mm, vias 0 -> 1
- net /ETH_TX_P: track 0.00 -> 45.8 mm, vias 0 -> 1
- net /SPI1_SCK: track 0.00 -> 39.4 mm, vias 0 -> 4
- net /SPI1_MOSI: track 0.00 -> 38.4 mm, vias 0 -> 4
- net /SPI2_SCK: track 0.00 -> 36.9 mm, vias 0 -> 2
- net /SPI2_MOSI: track 0.00 -> 34.0 mm, vias 0 -> 2
- net /USB_D-: track 0.00 -> 31.2 mm, vias 0 -> 2
- net /USB_D+: track 0.00 -> 31.0 mm, vias 0 -> 2
- net /SPI3_SCK: track 0.00 -> 24.6 mm
- net /MCO1: track 0.00 -> 24.0 mm, vias 0 -> 2
- net /SPI3_MOSI: track 0.00 -> 23.8 mm
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- added copper zone on F.Cu, net +3V3
- added copper zone on In2.Cu, net +3V3
- added copper zone on B.Cu, net +5V
- added copper zone on F.Cu, net +5V
- added copper zone on F.Cu, net +5V_DCDC
- added copper zone on F.Cu, net +5V_USB
- added copper zone on In2.Cu, net +5V_USB
- added copper zone on F.Cu, net /POE_V-
- added copper zone on F.Cu, net GND
- added copper zone on In1.Cu, net GND
- added copper zone on In2.Cu, net GND
- removed copper zone on In1.Cu, net (none)
- removed copper zone on In2.Cu, net (none)
Other:
- board text added: "FB2026"

Commit message: wip
Routing:
- net GND: track 73.3 -> 73.9 mm, vias 127 -> 129
- net /POE_V-: vias 0 -> 15
- net +5V_DCDC: vias 0 -> 5
- added copper zone on B.Cu, net +5V_DCDC
- added copper zone on B.Cu, net /POE_V-
- added copper zone on B.Cu, net GND

Commit message: wip
Parts:
- moved J3 33.1 mm to (123.5, 98.6), turned to -90 degrees
- moved R21 33.0 mm to (123.1, 125.3), turned to -90 degrees
- moved G*** 32.6 mm to (136.3, 106.3), turned to 0 degrees
- moved R4 32.0 mm to (124.1, 125.3), turned to -90 degrees
- moved SW2 31.7 mm to (123.6, 129.7), turned to -90 degrees
- moved D2 31.1 mm to (123.1, 123.4), turned to 90 degrees
- moved J10 30.2 mm to (155.2, 99.8), turned to 90 degrees
- moved D1 30.1 mm to (124.1, 123.4), turned to 90 degrees
- moved SW1 26.6 mm to (124.1, 104.8), turned to 0 degrees
- moved R1 23.3 mm to (129.0, 134.2)
- moved R2 23.3 mm to (126.1, 134.2)
- moved J1 23.3 mm to (127.7, 139.2)
- moved C17 22.8 mm to (123.5, 118.5)
- moved C11 22.8 mm to (124.1, 109.5)
- moved C58 22.8 mm to (131.6, 122.7)
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Connections:
- U10 pad 10: unconnected-(U10-PC2-Pad10) -> /LED_B
- U10 pad 14: /ETH_LED_0 -> /LED_A
- U10 pad 17: /ETH_RESET -> /SW0
- U10 pad 26: /SW0 -> unconnected-(U10-PB0-Pad26)
- U10 pad 27: /LED_B -> unconnected-(U10-PB1-Pad27)
- U10 pad 28: /LED_A -> unconnected-(U10-PB2-Pad28)
- U10 pad 35: unconnected-(U10-PB13-Pad35) -> /ETH_LED_0
- U10 pad 36: unconnected-(U10-PB14-Pad36) -> /ETH_RESET
Routing:
- net /ETH_TX_P: track 45.8 -> 15.5 mm, vias 1 -> 0
- net /ETH_RX_N: track 46.2 -> 15.9 mm, vias 1 -> 0
- net /ETH_RX_P: track 46.1 -> 15.8 mm, vias 1 -> 0
- net /ETH_TX_N: track 45.9 -> 15.7 mm, vias 1 -> 0
- net /SPI1_MOSI: track 38.6 -> 23.3 mm, vias 4 -> 0
- net /SPI1_SCK: track 39.4 -> 24.0 mm, vias 4 -> 0
- net Net-(J2-Pad14): track 5.14 -> 18.2 mm
- net +5V_DCDC: track 14.6 -> 2.59 mm
- net /MCO1: track 23.9 -> 12.6 mm
- net /SPI3_SCK: track 24.6 -> 34.5 mm, vias 0 -> 2
- net /SPI3_MOSI: track 23.8 -> 33.6 mm, vias 0 -> 2
- net Net-(J2-Pad12): track 16.7 -> 7.39 mm
- net /ETH_RESET: track 7.67 -> 16.4 mm, vias 0 -> 2
- net /SPI2_SCK: track 36.7 -> 28.0 mm
- net /RMII_TX_EN: track 6.73 -> 14.0 mm
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
Commit message: wip
Parts:
- added REF**: 4layer-flags-line, balto:4layer-flags-line, F.Cu at (121.5, 136.9)
- moved J10 0.14 mm to (155.1, 99.7)
Routing:
- net /RMII_RXD0: track 7.69 -> 14.5 mm
- net /RMII_RXD1: track 7.29 -> 13.7 mm
- net /RMII_CRS_DV: track 9.43 -> 12.1 mm
- net /USB_D+: track 30.8 -> 32.4 mm
- net /UART_TX: track 17.0 -> 15.8 mm
- net /POE_V+: track 21.9 -> 23.0 mm, vias 1 -> 6
- net /RMII_RX_ER: track 12.9 -> 12.2 mm
- net /RMII_REF_CLK: track 15.9 -> 15.3 mm
- net /USB_D-: track 31.8 -> 32.4 mm
- net GND: track 72.9 -> 72.8 mm, vias 118 -> 126
- added copper zone on B.Cu, net /POE_V+
- added copper zone on F.Cu, net /POE_V+

Commit message: wip
Parts:
- moved J1 0.58 mm to (128.3, 139.2)
- moved R1 0.58 mm to (129.6, 134.2)
- moved R2 0.58 mm to (126.7, 134.2)
- moved G*** 0.22 mm to (136.4, 106.1)
- moved REF** 0.20 mm to (121.7, 136.9)
