File: hardware/quakelight.kicad_sch (KiCad schematic)
At the start: 64 parts, among them J1 USB_C_Receptacle_USB2.0, J10 Conn_01x02_MountingPin, J2 RJ45_Abracon_ARJP11A-MASA-B-A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, J3 EZmate-4, J4 Conn_01x03_MountingPin, J5 Conn_01x03_MountingPin, J6 Conn_01x03_MountingPin, J7 TC2030-IDC-NL, SW1 SW_Push, SW2 SW_Push, U1 TPS7A0333DBVR, U10 STM32H573RIVx, U3 KSZ8081RNA, U4 SN74LV1T125DBV, U5 SN74LV1T125DBV, U6 TPS2116DRL, U7 SN74LV1T125DBV, Y1 25MHz, Y2 32.768kHz

Commit message: wip
Parts:
- removed C19: 100u, Capacitor_SMD:CP_Elec_6.3x7.7, symbol Device:C_Polarized
- removed J4, J5, J6: Conn_01x03_MountingPin, Connector_JST:JST_PH_S3B-PH-SM4-TB_1x03-1MP_P2.00mm_Horizontal, symbol Connector_Generic_MountingPin:Conn_01x03_MountingPin
- removed U4, U5, U7: SN74LV1T125DBV, Package_TO_SOT_SMD:SOT-23-5, symbol Logic_LevelTranslator:SN74LV1T125DBV
- added C14, C15, C16, C19, C23, C24, C25: 100u, Capacitor_SMD:C_1206_3216Metric, symbol Device:C
- added C20, C21, C22: 100n, balto:C_0402_Worthington, symbol Device:C
- added D3: SMAJ58A, Diode_SMD:D_SMA, symbol Diode:SMAJ58A
- added J4, J5, J9: PH, Connector_JST:JST_PH_S4B-PH-SM4-TB_1x04-1MP_P2.00mm_Horizontal, symbol Connector_Generic_MountingPin:Conn_01x04_MountingPin
- added R10, R11, R14, R15, R16, R8: 100, balto:R_0402_Worthington, symbol Device:R
- added R6: 0, balto:R_0402_Worthington, symbol Device:R
- added R7: 1k, balto:R_0402_Worthington, symbol Device:R
- added U4, U5, U8: SN74LVC2T45DCUR, Package_SO:VSSOP-8_2.3x2mm_P0.5mm, symbol Logic_LevelTranslator:SN74LVC2T45DCUR
- C13, C4, C8: value 10u -> 100u; footprint balto:C_0402_Worthington -> Capacitor_SMD:C_1206_3216Metric
Connections:
- net +3V3: now also SW1.2, C20.1, C21.1, C22.1, U4.1 (VCCA), U4.5 (DIR), U5.1 (VCCA), U5.5 (DIR), U8.1 (VCCA), U8.5 (DIR)
- net +5V: now also C14.1, C15.1, C16.1, J4.1 (Pin_1), J5.1 (Pin_1), J9.1 (Pin_1), U4.8 (VCCB), U5.8 (VCCB), U8.8 (VCCB)
- net +5V_DCDC: now also C19.1, C23.1, C24.1, C25.1
- net GND: now also C14.2, C15.2, C16.2, C19.2, C20.2, C21.2, C22.2, C23.2, C24.2, C25.2, J4.4 (Pin_4), J4.MP (MountPin), J5.4 (Pin_4), J5.MP (MountPin), J9.4 (Pin_4), J9.MP (MountPin), R7.2, U4.4 (GND), U5.4 (GND), U8.4 (GND); no longer SW1.2, U10.62 (BOOT0)
- net POE_V+: now also D3.1 (A1)
- net POE_V-: now also D3.2 (A2)
- net SPI1_MOSI: now also U8.3 (A2)
- net SPI2_MOSI: now also U4.3 (A2)
- net SPI3_MOSI: now also U5.3 (A2)
- net SW1: now also U10.63 (PB8), R6.1; no longer SW1.1
- net SPI2_SCK: now reaches U10.45 (PA9)
- net SPI2_SCK: now also U4.2 (A1)
- net SPI3_SCK: now reaches U10.54 (PC10)
- net SPI3_SCK: now also U5.2 (A1)
- net SPI1_SCK: now reaches U10.57 (PB3(JTDO)
- net SPI1_SCK: now also U8.2 (A1)
- new net: R14.2, U4.6 (B2)
- new net: R11.2, U4.7 (B1)
- new net: J9.2 (Pin_2), R8.1
- new net: R8.2, U8.7 (B1)
- new net: J4.3 (Pin_3), R14.1
- new net: R10.2, U8.6 (B2)
- new net: J5.3 (Pin_3), R16.1
- new net: R16.2, U5.6 (B2)
- new net: J4.2 (Pin_2), R11.1
- new net: J9.3 (Pin_3), R10.1
- new net: J5.2 (Pin_2), R15.1
- new net: R15.2, U5.7 (B1)
- new net BOOT0: R6.2, R7.1, SW1.1, U10.62 (BOOT0)
- no-connect marks 33 -> 29
Other:
- note removed: "spi1 sck reserve"
- note removed: "spi2 sck reserve"
- note removed: "spi3 sck reserve"
- moved on the sheet: C18, C3, C4, C5, C64, C66, C67, C68, C69, D1, D2, J10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

Commit message: wip
Parts:
- added C26, C27: 1u, balto:C_0402_Worthington, symbol Device:C
- R12: value 75k -> 36k
- R5: value 75k -> 0; footprint balto:R_0402_Worthington -> Resistor_SMD:R_0805_2012Metric
Connections:
- net +5V_DCDC: now also C27.1; no longer R5.1
- net +5V_USB: now also C26.1
- net ETH_INT: now also U10.22 (PA6); no longer U10.17 (PA3)
- net ETH_LED_0: now also U10.14 (PA0)
- net ETH_RESET: now also U10.17 (PA3); no longer U10.8 (PC0)
- net GND: now also R5.2, C26.2, C27.2; no longer J2.SH
- net LED_A: now also U10.28 (PB2)
- net LED_B: now also U10.27 (PB1)
- net SW0: now also U10.26 (PB0)
- net at R12.2, R13.1, U6.4 (PR1): no longer R5.2
- new net: J2.SH, R5.1
- no-connect marks 29 -> 24
Other:
- note added: "|-----length match-----|"
- moved on the sheet: C18, C19, C23, C24, C25, C3, C64, C66, C67, C68, C69, D1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

Commit message: wip
Connections:
- net ETH_LED_0: now also U10.35 (PB13); no longer U10.14 (PA0)
- net ETH_RESET: now also U10.36 (PB14); no longer U10.17 (PA3)
- net LED_A: now also U10.14 (PA0); no longer U10.28 (PB2)
- net LED_B: now also U10.10 (PC2); no longer U10.27 (PB1)
- net SW0: now also U10.17 (PA3); no longer U10.26 (PB0)
- no-connect marks 24 -> 21

Commit message: wip
Other:
- note added: "|---length match---|"
- note removed: "|-----length match-----|"

Commit message: wip
Connections:
- no-connect marks 21 -> 27

Commit message: hw: move output on separate sheet
Parts:
- removed C10, C20, C21, C22, C5, C6: 100n, balto:C_0402_Worthington, symbol Device:C
- removed C13, C14, C15, C16, C4, C8: 100u, Capacitor_SMD:C_1206_3216Metric, symbol Device:C
- removed J4, J5, J9: PH, Connector_JST:JST_PH_S4B-PH-SM4-TB_1x04-1MP_P2.00mm_Horizontal, symbol Connector_Generic_MountingPin:Conn_01x04_MountingPin
- removed R10, R11, R14, R15, R16, R8: 100, balto:R_0402_Worthington, symbol Device:R
- removed U4, U5, U8: SN74LVC2T45DCUR, Package_SO:VSSOP-8_2.3x2mm_P0.5mm, symbol Logic_LevelTranslator:SN74LVC2T45DCUR
Other:
- added sheet Output_1 (led_output.kicad_sch)
- added sheet Output_2 (led_output.kicad_sch)
- added sheet Output_3 (led_output.kicad_sch)

Commit message: hw: add few notes
Other:
- note added: "TODO: cap"
- note added: "TODO: filters"
- note added: "TODO: review decoupling"

Commit message: hw: dnp update
Parts:
- C23, C25: now fitted
